File: panel/panel.kicad_pcb (KiCad board)
At the start: 2 copper layers, 70.8 x 128.5 mm, 4 parts

Commit message: Changed inputs to circles on panels
Changed lines of the file:
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@@
   (gr_rect (start 38 124.15) (end 38.2 124.55) (layer "F.SilkS") (width 0.01) (fill solid))
   (gr_rect (start 40.6 124.95) (end 40.8 125.35) (layer "F.SilkS") (width 0.01) (fill solid))
+  (gr_rect (start 44.625 15.75) (end 53.625 25.75) (layer "F.SilkS") (width 0.15) (fill solid))
   (gr_rect (start 32.2 123.35) (end 32.4 123.75) (layer "F.SilkS") (width 0.01) (fill solid))
   (gr_rect (start 30.8 124.15) (end 31 124.55) (layer "F.SilkS") (width 0.01) (fill solid))
@@
   (gr_rect (start 41 125.35) (end 41.2 125.75) (layer "F.SilkS") (width 0.01) (fill solid))
   (gr_rect (start 32.6 124.15) (end 32.8 124.55) (layer "F.SilkS") (width 0.01) (fill solid))
-  (gr_circle (center 21.625 20.75) (end 26.625 20.75) (layer "F.SilkS") (width 0.15) (fill solid))
   (gr_rect (start 37 124.55) (end 37.2 124.95) (layer "F.SilkS") (width 0.01) (fill solid))
   (gr_rect (start 35.4 124.95) (end 35.6 125.35) (layer "F.SilkS") (width 0.01) (fill solid))
@@
   (gr_rect (start 33 125.75) (end 33.2 126.15) (layer "F.SilkS") (width 0.01) (fill solid))
   (gr_rect (start 42 125.75) (end 42.2 126.15) (layer "F.SilkS") (width 0.01) (fill solid))
-  (gr_circle (center 49.125 20.75) (end 54.125 20.75) (layer "F.SilkS") (width 0.15) (fill solid))
   (gr_rect (start 37.8 124.95) (end 38 125.35) (layer "F.SilkS") (width 0.01) (fill solid))
   (gr_rect (start 39 123.35) (end 39.2 123.75) (layer "F.SilkS") (width 0.01) (fill solid))
@@
   (gr_rect (start 45.8 123.75) (end 46 124.15) (layer "F.SilkS") (width 0.01) (fill solid))
   (gr_line (start 5.9 90.3) (end 23 90.3) (layer "F.SilkS") (width 0.5))
+  (gr_rect (start 17.25 15.75) (end 26.25 25.75) (layer "F.SilkS") (width 0.15) (fill solid))
   (gr_rect (start 45.4 123.35) (end 45.6 123.75) (layer "F.SilkS") (width 0.01) (fill solid))
   (gr_rect (start 27.8 125.75) (end 28 126.15) (layer "F.SilkS") (width 0.01) (fill solid))
